Commit message: setting up simulation, adding bigger map

File: workspace/src/wheelchair_description/urdf/wheelchair_gazebo.xacro (robot description, xacro)
@@ -5,5 +5,5 @@
     <plugin name="differential_drive_controller" filename="libgazebo_ros_diff_drive.so">
       <alwaysOn>true</alwaysOn>
-      <commandTopic>diff/cmd_vel</commandTopic>
+      <commandTopic>wheelchair_diff/cmd_vel</commandTopic>
       <odometryTopic>odom</odometryTopic>
       <odometryFrame>odom</odometryFrame>
@@ -81,5 +81,5 @@
     <material>Gazebo/Grey</material>
   </gazebo>
-  <gazebo reference="rplidar">
+  <!-- <gazebo reference="rplidar">
     <material>Gazebo/DarkGrey</material>
     <sensor type="gpu_ray" name="head_rplidar_sensor">
@@ -103,4 +103,40 @@
         <noise>
           <type>gaussian</type>
+          < Noise parameters based on published spec for Hokuyo laser
+               achieving "+-30mm" accuracy at range < 10m.  A mean of 0.0m and
+               stddev of 0.01m will put 99.7% of samples within 0.03m of the true
+               reading. >
+          <mean>0.0</mean>
+          <stddev>0.01</stddev>
+        </noise>
+      </ray>
+      <plugin name="gazebo_ros_head_rplidar_controller" filename="libgazebo_ros_gpu_laser.so">
+        <topicName>scan</topicName>
+        <frameName>rplidar</frameName>
+      </plugin>
+    </sensor>
+  </gazebo> -->
+  <gazebo reference="rplidar">
+    <material>Gazebo/DarkGrey</material>
+    <sensor type="gpu_ray" name="head_rplidar_sensor">
+      <pose>0 0 0 0 0 0</pose>
+      <visualize>true</visualize>
+      <update_rate>15</update_rate>
+      <ray>
+        <scan>
+          <horizontal>
+            <samples>720</samples>
+            <resolution>1</resolution>
+            <min_angle>-3.14</min_angle>
+            <max_angle>3.14</max_angle>
+          </horizontal>
+        </scan>
+        <range>
+          <min>0.1</min>
+          <max>25.0</max>
+          <resolution>0.01</resolution>
+        </range>
+        <noise>
+          <type>gaussian</type>
           <!-- Noise parameters based on published spec for Hokuyo laser
                achieving "+-30mm" accuracy at range < 10m.  A mean of 0.0m and
@@ -112,5 +148,5 @@
       </ray>
       <plugin name="gazebo_ros_head_rplidar_controller" filename="libgazebo_ros_gpu_laser.so">
-        <topicName>scan</topicName>
+        <topicName>scan_raw</topicName>
         <frameName>rplidar</frameName>
       </plugin>

File: workspace/src/wheelchair_description/urdf/wheelchair_real_new.xacro (robot description, xacro)
@@ -174,6 +174,7 @@
                type="fixed"
                axis_xyz="0 0 0"
-               origin_rpy="0 0 -1.57" origin_xyz="0.23 0 -0.15"
+               origin_rpy="0 0 0" origin_xyz="0.23 0 -0.15"
                parent="chassis" child="rplidar" />
+               <!-- origin_rpy="0 0 -1.57" origin_xyz="0.23 0 -0.15" -->
 <!--Real_Sense-->
     <!--D435 with tilted angle as in real wheelchair-->
